File: RaspberryPiProtoHat.kicad_pcb (KiCad board)
At the start: 2 copper layers, 65 x 56 mm, 134 parts, among them J1 Conn_01x02_Male, J2 Conn_01x02_Male, J3 Conn_01x24_Female, J4 Conn_01x09_Female, J5 Conn_01x09_Female, J6 Conn_01x21_Female, P1 Conn_02x20_Odd_Even, Q1 Q_NPN_BCE, SW1 SW_Push

Commit message: Updated bypass capacitors to 1206 footprint for ease of soldering and added BOM
Parts:
- C1, C2: footprint Capacitor_SMD:C_0603_1608Metric -> Capacitor_SMD:C_1206_3216Metric
- moved C2 4.70 mm to (206.6, 110.5)
- moved C1 2.22 mm to (202.8, 108.9)
Routing:
- net +3V3: track 81.8 -> 77.3 mm
- net +5V: track 100.5 -> 104.4 mm
- net GND: track 159.7 -> 163.5 mm

Commit message: Version 2.0
Parts:
- MK1, MK2, MK3, MK4, MK5, MK6, MK7, MK8: footprint MountingHole:MountingHole_2.7mm_M2.5 -> MountingHole:MountingHole_3.2mm_M3
- moved MK8 0.31 mm to (234.8, 115.2)
- moved MK5 0.18 mm to (210.7, 115.2)
- moved MK7 0.18 mm to (210.7, 139.3)
- moved MK6 0.16 mm to (234.5, 139.3)
